File: lighting.sch (KiCad schematic (older format))
At the start: 6 parts

Commit message: I have no idea what I'm doing dot jpg
Parts:
- C1: renamed from C?; footprint (none) -> Capacitors_ThroughHole:C_Disc_D7.5_P5
- IC1: renamed from IC?; footprint DIP8 -> MCU-ATTINY85-20PU_DIP8_:DIP254P762X533-8
- P1: renamed from P?; value CONN_01X04 -> LDP8806; footprint (none) -> Pin_Headers:Pin_Header_Straight_1x04
- P2: renamed from P?; value CONN_02X03 -> SPI; footprint (none) -> Pin_Headers:Pin_Header_Straight_2x03
- R1: renamed from R?; footprint (none) -> Resistors_ThroughHole:Resistor_Vertical_RM5mm
- SW1: renamed from SW?; footprint (none) -> Buttons_Switches_ThroughHole:SW_PUSH_SMALL
Connections:
- wire segments 26 -> 30
Other:
- moved on the sheet: C1, IC1, P1, P2, R1, SW1
