File: lumos.sch (KiCad schematic (older format))
At the start: 6 parts, among them IC1 ATTINY85-P, P1 LDP8806, P2 SPI, SW1 SW_PUSH

Commit message: Near final layout of the lumos 0.1a board.
Parts:
- added CON1: BARREL_JACK, Connect:BARREL_JACK, symbol BARREL_JACK
Connections:
- wire segments 30 -> 39
Other:
- moved on the sheet: R1, SW1
Changed lines of the file:
@@
 LIBS:contrib
 LIBS:valves
-LIBS:lighting-cache
+LIBS:MCU-ATTINY85-20PU_DIP8_
+LIBS:lumos-cache
 EELAYER 25 0
 EELAYER END
@@
 $EndComp
 $Comp
-L GND #PWR01
+L GND #PWR10
 U 1 1 56AEEB24
 P 7050 4200
-F 0 "#PWR01" H 7050 3950 50  0001 C CNN
+F 0 "#PWR10" H 7050 3950 50  0001 C CNN
 F 1 "GND" H 7050 4050 50  0000 C CNN
 F 2 "" H 7050 4200 50  0000 C CNN
@@
 $EndComp
 $Comp
-L +5V #PWR02
+L +5V #PWR9
 U 1 1 56AEEB40
 P 7050 3300
-F 0 "#PWR02" H 7050 3150 50  0001 C CNN
+F 0 "#PWR9" H 7050 3150 50  0001 C CNN
 F 1 "+5V" H 7050 3440 50  0000 C CNN
 F 2 "" H 7050 3300 50  0000 C CNN
@@
 MOSI
 $Comp
-L GND #PWR03
+L GND #PWR6
 U 1 1 56AEEE75
 P 4950 4950
-F 0 "#PWR03" H 4950 4700 50  0001 C CNN
+F 0 "#PWR6" H 4950 4700 50  0001 C CNN
 F 1 "GND" H 4950 4800 50  0000 C CNN
 F 2 "" H 4950 4950 50  0000 C CNN
@@
 $EndComp
 $Comp
-L +5V #PWR04
+L +5V #PWR5
 U 1 1 56AEEE91
 P 4950 4450
-F 0 "#PWR04" H 4950 4300 50  0001 C CNN
+F 0 "#PWR5" H 4950 4300 50  0001 C CNN
 F 1 "+5V" H 4950 4590 50  0000 C CNN
 F 2 "" H 4950 4450 50  0000 C CNN
@@
 $EndComp
 $Comp
-L +5V #PWR05
+L +5V #PWR2
 U 1 1 56AEEEB1
-P 6400 4500
-F 0 "#PWR05" H 6400 4350 50  0001 C CNN
-F 1 "+5V" H 6400 4640 50  0000 C CNN
-F 2 "" H 6400 4500 50  0000 C CNN
-F 3 "" H 6400 4500 50  0000 C CNN
-	1    6400 4500
-	1    0    0    -1
-$EndComp
-$Comp
-L GND #PWR06
+P 3050 4850
+F 0 "#PWR2" H 3050 4700 50  0001 C CNN
+F 1 "+5V" H 3050 4990 50  0000 C CNN
+F 2 "" H 3050 4850 50  0000 C CNN
+F 3 "" H 3050 4850 50  0000 C CNN
+	1    3050 4850
+	1    0    0    -1
+$EndComp
+$Comp
+L GND #PWR1
 U 1 1 56AEEED5
-P 7000 5150
-F 0 "#PWR06" H 7000 4900 50  0001 C CNN
-F 1 "GND" H 7000 5000 50  0000 C CNN
-F 2 "" H 7000 5150 50  0000 C CNN
-F 3 "" H 7000 5150 50  0000 C CNN
-	1    7000 5150
-	1    0    0    -1
+P 2450 5500
+F 0 "#PWR1" H 2450 5250 50  0001 C CNN
+F 1 "GND" H 2450 5350 50  0000 C CNN
+F 2 "" H 2450 5500 50  0000 C CNN
+F 3 "" H 2450 5500 50  0000 C CNN
+	1    2450 5500
+	-1   0    0    -1
 $EndComp
 $Comp
 L SW_PUSH SW1
 U 1 1 56AEEEF1
-P 6700 5000
-F 0 "SW1" H 6850 5110 50  0000 C CNN
-F 1 "SW_PUSH" H 6700 4920 50  0000 C CNN
-F 2 "Buttons_Switches_ThroughHole:SW_PUSH_SMALL" H 6700 5000 50  0001 C CNN
-F 3 "" H 6700 5000 50  0000 C CNN
-	1    6700 5000
-	1    0    0    -1
+P 2750 5350
+F 0 "SW1" H 2900 5460 50  0000 C CNN
+F 1 "SW_PUSH" H 2750 5270 50  0000 C CNN
+F 2 "Buttons_Switches_ThroughHole:SW_PUSH_SMALL" H 2750 5350 50  0001 C CNN
+F 3 "" H 2750 5350 50  0000 C CNN
+	1    2750 5350
+	-1   0    0    -1
 $EndComp
 $Comp
 L R R1
 U 1 1 56AEEF7F
-P 6400 4750
-F 0 "R1" V 6480 4750 50  0000 C CNN
-F 1 "10k" V 6400 4750 50  0000 C CNN
-F 2 "Resistors_ThroughHole:Resistor_Vertical_RM5mm" V 6330 4750 50  0001 C CNN
-F 3 "" H 6400 4750 50  0000 C CNN
-	1    6400 4750
-	1    0    0    -1
-$EndComp
-Text Label 6200 5250 0    60   ~ 0
+P 3050 5100
+F 0 "R1" V 3130 5100 50  0000 C CNN
+F 1 "10k" V 3050 5100 50  0000 C CNN
+F 2 "Resistors_ThroughHole:Resistor_Vertical_RM5mm" V 2980 5100 50  0001 C CNN
+F 3 "" H 3050 5100 50  0000 C CNN
+	1    3050 5100
+	-1   0    0    -1
+$EndComp
+Text Label 3250 5600 2    60   ~ 0
 RST
 Text Label 3000 3700 0    60   ~ 0
-CLK0
+SCK
 Text Label 3000 3800 0    60   ~ 0
-MISO
+MOSI
 Wire Wire Line
 	4150 4000 3850 4000
 Wire Wire Line
-	4150 3500 3850 3500
-Wire Wire Line
-	4150 3600 3850 3600
-Wire Wire Line
-	4150 3700 3850 3700
+	3550 3500 4150 3500
+Wire Wire Line
+	3700 3600 4150 3600
+Wire Wire Line
+	2900 3700 4150 3700
 Wire Wire Line
 	4150 3800 3850 3800
@@
 Connection ~ 6900 4000
 Wire Wire Line
-	4250 4600 4050 4600
-Wire Wire Line
-	4250 4700 4050 4700
-Wire Wire Line
-	4250 4800 4050 4800
+	3700 4600 4250 4600
+Wire Wire Line
+	3450 4700 4250 4700
+Wire Wire Line
+	3850 4800 4250 4800
 Wire Wire Line
 	4750 4700 5150 4700
@@
 	4950 4800 4950 4950
 Wire Wire Line
-	6400 4900 6400 5250
-Wire Wire Line
-	6400 4600 6400 4500
-Wire Wire Line
-	7000 5000 7000 5150
-Wire Wire Line
-	6400 5250 6200 5250
-Connection ~ 6400 5000
-Wire Wire Line
-	2900 3700 3250 3700
-Wire Wire Line
-	2900 3800 3250 3800
+	3050 5250 3050 5750
+Wire Wire Line
+	3050 4950 3050 4850
+Wire Wire Line
+	2450 5350 2450 5500
+Connection ~ 3050 5350
+Wire Wire Line
+	2900 3800 3550 3800
 Wire Wire Line
 	2900 3600 3200 3600
@@
 	3200 3900 3200 4150
 $Comp
-L GND #PWR07
+L GND #PWR4
 U 1 1 56AEF722
 P 3200 4150
-F 0 "#PWR07" H 3200 3900 50  0001 C CNN
+F 0 "#PWR4" H 3200 3900 50  0001 C CNN
 F 1 "GND" H 3200 4000 50  0000 C CNN
 F 2 "" H 3200 4150 50  0000 C CNN
@@
 $EndComp
 $Comp
-L +5V #PWR08
+L +5V #PWR3
 U 1 1 56AEF7EA
 P 3200 3350
-F 0 "#PWR08" H 3200 3200 50  0001 C CNN
+F 0 "#PWR3" H 3200 3200 50  0001 C CNN
 F 1 "+5V" H 3200 3490 50  0000 C CNN
 F 2 "" H 3200 3350 50  0000 C CNN
@@
 	1    0    0    -1
 $EndComp
+Wire Wire Line
+	3550 3500 3550 4300
+Wire Wire Line
+	5150 4700 5150 4300
+Wire Wire Line
+	5150 4300 3550 4300
+Connection ~ 3550 3800
+Wire Wire Line
+	3700 4600 3700 3600
+Wire Wire Line
+	3450 4700 3450 3700
+Connection ~ 3450 3700
+Wire Wire Line
+	3850 4000 3850 5750
+Connection ~ 3850 4800
+Wire Wire Line
+	3850 5750 3050 5750
+$Comp
+L BARREL_JACK CON1
+U 1 1 56B423CF
+P 5100 5700
+F 0 "CON1" H 5100 5950 50  0000 C CNN
+F 1 "BARREL_JACK" H 5100 5500 50  0000 C CNN
+F 2 "Connect:BARREL_JACK" H 5100 5700 50  0001 C CNN
+F 3 "" H 5100 5700 50  0000 C CNN
+	1    5100 5700
+	1    0    0    -1
+$EndComp
+Wire Wire Line
+	5400 5800 5600 5800
+Wire Wire Line
+	5600 5800 5600 5900
+Wire Wire Line
+	5400 5600 5600 5600
+Wire Wire Line
+	5600 5600 5600 5500
+$Comp
+L GND #PWR8
+U 1 1 56B42566
+P 5600 5900
+F 0 "#PWR8" H 5600 5650 50  0001 C CNN
+F 1 "GND" H 5600 5750 50  0000 C CNN
+F 2 "" H 5600 5900 50  0000 C CNN
+F 3 "" H 5600 5900 50  0000 C CNN
+	1    5600 5900
+	1    0    0    -1
+$EndComp
+$Comp
+L +5V #PWR7
+U 1 1 56B42588
+P 5600 5500
+F 0 "#PWR7" H 5600 5350 50  0001 C CNN
+F 1 "+5V" H 5600 5640 50  0000 C CNN
+F 2 "" H 5600 5500 50  0000 C CNN
+F 3 "" H 5600 5500 50  0000 C CNN
+	1    5600 5500
+	1    0    0    -1
+$EndComp

Commit message: PCB w/ traces, silk screening, updated ground on barrel jack
Connections:
- net GND: now also CON1.3
Changed lines of the file:
@@
 	5400 5800 5600 5800
 Wire Wire Line
-	5600 5800 5600 5900
+	5600 5700 5600 5900
 Wire Wire Line
 	5400 5600 5600 5600
@@
 	1    0    0    -1
 $EndComp
+Wire Wire Line
+	5400 5700 5600 5700
+Connection ~ 5600 5800
 $EndSCHEMATC
